File: pcb/blinker.kicad_pcb (KiCad board)
At the start: 2 copper layers, 50.8 x 50.8 mm, 14 parts, among them J1 ISP, U1 ATtiny10-TS

Commit message: About to route PCB.
Parts:
- D2: footprint Diode_SMD:D_SOD-123 -> Diode_SMD:D_SOD-123F
- renumbered C4 to C1, C3 to C2, C2 to C3, C1 to C4, C6 to C5, C5 to C6
Other:
- board text added: "CAP PWR"
- board text added: "ISP"
- board text added: "SOL PNL"
Changed lines of the file:
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@@
   (net 11 "5VCC")
   (net 12 "LED")
-  (footprint "Diode_SMD:D_SOD-123" (layer "F.Cu")
+  (footprint "Diode_SMD:D_SOD-123F" (layer "F.Cu")
     (at 165.315 94.425 180)
-    (descr "SOD-123")
-    (tags "SOD-123")
-    (property "LCSC" "C707156")
+    (descr "D_SOD-123F")
+    (tags "D_SOD-123F")
+    (property "LCSC" "C362294")
     (property "Sheetfile" "blinker.kicad_sch")
     (property "Sheetname" "")
     (attr smd)
-    (fp_text reference "D2" (at 0 -2 180) (layer "F.SilkS")
+    (fp_text reference "D2" (at 0.005 2.245 180) (layer "F.SilkS")
       (effects (font (size 1 1) (thickness 0.15)))
     )
@@
       (effects (font (size 1 1) (thickness 0.15)))
     )
-    (fp_text user "${REFERENCE}" (at 0 -2 180) (layer "F.Fab")
+    (fp_text user "${REFERENCE}" (at -0.127 -1.905 180) (layer "F.Fab")
       (effects (font (size 1 1) (thickness 0.15)))
     )
-    (fp_line (start -2.25 -1) (end 1.65 -1) (layer "F.SilkS") (width 0.12))
-    (fp_line (start -2.25 -1) (end -2.25 1) (layer "F.SilkS") (width 0.12))
-    (fp_line (start -2.25 1) (end 1.65 1) (layer "F.SilkS") (width 0.12))
-    (fp_line (start -2.35 -1.15) (end -2.35 1.15) (layer "F.CrtYd") (width 0.05))
-    (fp_line (start 2.35 -1.15) (end 2.35 1.15) (layer "F.CrtYd") (width 0.05))
-    (fp_line (start -2.35 -1.15) (end 2.35 -1.15) (layer "F.CrtYd") (width 0.05))
-    (fp_line (start 2.35 1.15) (end -2.35 1.15) (layer "F.CrtYd") (width 0.05))
+    (fp_line (start -2.2 -1) (end -2.2 1) (layer "F.SilkS") (width 0.12))
+    (fp_line (start -2.2 1) (end 1.65 1) (layer "F.SilkS") (width 0.12))
+    (fp_line (start -2.2 -1) (end 1.65 -1) (layer "F.SilkS") (width 0.12))
+    (fp_line (start -2.2 -1.15) (end -2.2 1.15) (layer "F.CrtYd") (width 0.05))
+    (fp_line (start 2.2 -1.15) (end 2.2 1.15) (layer "F.CrtYd") (width 0.05))
+    (fp_line (start 2.2 1.15) (end -2.2 1.15) (layer "F.CrtYd") (width 0.05))
+    (fp_line (start -2.2 -1.15) (end 2.2 -1.15) (layer "F.CrtYd") (width 0.05))
+    (fp_line (start 0.25 0.4) (end -0.35 0) (layer "F.Fab") (width 0.1))
+    (fp_line (start -0.35 0) (end 0.25 -0.4) (layer "F.Fab") (width 0.1))
     (fp_line (start -0.35 0) (end -0.35 -0.55) (layer "F.Fab") (width 0.1))
+    (fp_line (start -0.35 0) (end -0.35 0.55) (layer "F.Fab") (width 0.1))
     (fp_line (start -0.75 0) (end -0.35 0) (layer "F.Fab") (width 0.1))
+    (fp_line (start -1.4 -0.9) (end 1.4 -0.9) (layer "F.Fab") (width 0.1))
+    (fp_line (start 0.25 -0.4) (end 0.25 0.4) (layer "F.Fab") (width 0.1))
+    (fp_line (start 0.25 0) (end 0.75 0) (layer "F.Fab") (width 0.1))
     (fp_line (start 1.4 -0.9) (end 1.4 0.9) (layer "F.Fab") (width 0.1))
-    (fp_line (start -0.35 0) (end -0.35 0.55) (layer "F.Fab") (width 0.1))
+    (fp_line (start 1.4 0.9) (end -1.4 0.9) (layer "F.Fab") (width 0.1))
     (fp_line (start -1.4 0.9) (end -1.4 -0.9) (layer "F.Fab") (width 0.1))
-    (fp_line (start -1.4 -0.9) (end 1.4 -0.9) (layer "F.Fab") (width 0.1))
-    (fp_line (start 0.25 0) (end 0.75 0) (layer "F.Fab") (width 0.1))
-    (fp_line (start 0.25 0.4) (end -0.35 0) (layer "F.Fab") (width 0.1))
-    (fp_line (start 1.4 0.9) (end -1.4 0.9) (layer "F.Fab") (width 0.1))
-    (fp_line (start 0.25 -0.4) (end 0.25 0.4) (layer "F.Fab") (width 0.1))
-    (fp_line (start -0.35 0) (end 0.25 -0.4) (layer "F.Fab") (width 0.1))
-    (pad "1" smd rect (at -1.65 0 180) (size 0.9 1.2) (layers "F.Cu" "F.Paste" "F.Mask")
+    (pad "1" smd rect (at -1.4 0 180) (size 1.1 1.1) (layers "F.Cu" "F.Paste" "F.Mask")
       (net 9 "2.7VCC") (pinfunction "K") (pintype "passive"))
-    (pad "2" smd rect (at 1.65 0 180) (size 0.9 1.2) (layers "F.Cu" "F.Paste" "F.Mask")
+    (pad "2" smd rect (at 1.4 0 180) (size 1.1 1.1) (layers "F.Cu" "F.Paste" "F.Mask")
       (net 2 "GND") (pinfunction "A") (pintype "passive"))
-    (model "${KICAD6_3DMODEL_DIR}/Diode_SMD.3dshapes/D_SOD-123.wrl"
+    (model "${KICAD6_3DMODEL_DIR}/Diode_SMD.3dshapes/D_SOD-123F.wrl"
       (offset (xyz 0 0 0))
       (scale (xyz 1 1 1))
@@
     (property "Sheetname" "")
     (attr through_hole)
-    (fp_text reference "C2" (at 3.75 9.25 60) (layer "B.SilkS")
+    (fp_text reference "C3" (at 3.75 9.25 60) (layer "B.SilkS")
       (effects (font (size 1 1) (thickness 0.15)) (justify mirror))
     )
@@
     (property "Sheetname" "")
     (attr through_hole)
-    (fp_text reference "C4" (at 3.75 9.25) (layer "B.SilkS")
+    (fp_text reference "C1" (at 3.75 9.25) (layer "B.SilkS")
       (effects (font (size 1 1) (thickness 0.15)) (justify mirror))
     )
@@
     (property "Sheetname" "")
     (attr through_hole)
-    (fp_text reference "C5" (at 3.75 9.25 60) (layer "B.SilkS")
+    (fp_text reference "C6" (at 3.75 9.25 60) (layer "B.SilkS")
       (effects (font (size 1 1) (thickness 0.15)) (justify mirror))
     )
@@
     (property "Sheetname" "")
     (attr through_hole)
-    (fp_text reference "C3" (at 3.75 9.25 120) (layer "B.SilkS")
+    (fp_text reference "C2" (at 3.75 9.25 120) (layer "B.SilkS")
       (effects (font (size 1 1) (thickness 0.15)) (justify mirror))
     )
@@
     (property "Sheetname" "")
     (attr through_hole)
-    (fp_text reference "C6" (at 3.75 9.25 120) (layer "B.SilkS")
+    (fp_text reference "C5" (at 3.75 9.25 120) (layer "B.SilkS")
       (effects (font (size 1 1) (thickness 0.15)) (justify mirror))
     )
@@
     (property "Sheetname" "")
     (attr through_hole)
-    (fp_text reference "C1" (at 5.775 8.355) (layer "B.SilkS")
+    (fp_text reference "C4" (at 5.775 8.355) (layer "B.SilkS")
       (effects (font (size 1 1) (thickness 0.15)) (justify mirror))
     )
@@
   (gr_circle (center 125.66 42.17) (end 125.66 42.17) (layer "F.Cu") (width 0.2) (fill none))
   (gr_circle (center 165.1 101.6) (end 190.5 101.6) (layer "Edge.Cuts") (width 0.2) (fill none))
+  (gr_text "SOL\nPNL" (at 161.99 98.41 270) (layer "B.SilkS")
+    (effects (font (size 1.5 1.5) (thickness 0.3)) (justify mirror))
+  )
+  (gr_text "CAP\nPWR" (at 164.11 103.37) (layer "B.SilkS")
+    (effects (font (size 1.5 1.5) (thickness 0.3)) (justify mirror))
+  )
+  (gr_text "ISP" (at 167.71 95.6 90) (layer "B.SilkS")
+    (effects (font (size 1.5 1.5) (thickness 0.3)) (justify mirror))
+  )
 )

Commit message: Routed
Parts:
- moved D2 21.7 mm to (146.7, 105.5)
- moved D1 12.4 mm to (158.1, 92.7), turned to -90 degrees
- moved J1 10.4 mm to (170.8, 106.9), turned to 0 degrees
- moved R1 8.78 mm to (164.5, 94.1), turned to 90 degrees
- moved D3 2.53 mm to (165.3, 80.9)
- moved U1 1.45 mm to (164.7, 99.9), turned to 180 degrees
- moved JP1 0.37 mm to (163.2, 107.4)
- moved SC1 0.09 mm to (158.1, 97.6)
Connections:
- net Net-(D1-Pad2) renamed /SLR_IN
- net Net-(D3-Pad1) renamed /LED_R
Routing:
- net GND: track 0.00 -> 51.3 mm
- net 5VCC: track 0.00 -> 49.8 mm, vias 0 -> 1
- net 2.7VCC: track 0.00 -> 18.0 mm
- net /LED_R: track 0.00 -> 12.4 mm
- net RESET: track 0.00 -> 9.04 mm, vias 0 -> 1
- net TPIDATA: track 0.00 -> 8.13 mm
- net TPICLK: track 0.00 -> 5.11 mm
- net LED: track 0.00 -> 4.38 mm
- net /SLR_IN: track 0.00 -> 3.77 mm

Commit message: routed.
Routing:
- net GND: track 51.3 -> 5.32 mm
- net 2.7VCC: track 18.0 -> 34.3 mm
- added copper zone on B.Cu, net 2.7VCC
- added copper zone on F.Cu, net GND
Other:
- board size 50.8 x 50.8 mm -> 55.9 x 55.9 mm
