File: pcb/blinker.kicad_sch (KiCad schematic)
At the start: 41 parts, among them J1 ISP, U1 ATtiny10-TS, U2 M24C01-FDW

Commit message: PCB footprint fixes. Still wrong data bus direction.
Parts:
- C18: value 120 pF -> 120pF
- D10, D11, D12, D13, D14, D15, D16, D2, D3, D4, D5, D6, D7, D8, D9: value WS2812B -> LED
Changed lines of the file:
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@@
 			)
 		)
-		(property "Value" "WS2812B"
+		(property "Value" "LED"
 			(at 243.84 74.5646 90)
 			(effects
@@
 			)
 		)
-		(property "Value" "WS2812B"
+		(property "Value" "LED"
 			(at 220.98 56.7846 90)
 			(effects
@@
 			)
 		)
-		(property "Value" "WS2812B"
+		(property "Value" "LED"
 			(at 220.98 110.1246 90)
 			(effects
@@
 			)
 		)
-		(property "Value" "WS2812B"
+		(property "Value" "LED"
 			(at 220.98 39.0046 90)
 			(effects
@@
 			)
 		)
-		(property "Value" "WS2812B"
+		(property "Value" "LED"
 			(at 267.97 56.7846 90)
 			(effects
@@
 			)
 		)
-		(property "Value" "WS2812B"
+		(property "Value" "LED"
 			(at 267.97 110.1246 90)
 			(effects
@@
 			)
 		)
-		(property "Value" "WS2812B"
+		(property "Value" "LED"
 			(at 243.84 56.7846 90)
 			(effects
@@
 			)
 		)
-		(property "Value" "WS2812B"
+		(property "Value" "LED"
 			(at 220.98 74.5646 90)
 			(effects
@@
 			)
 		)
-		(property "Value" "WS2812B"
+		(property "Value" "LED"
 			(at 243.84 110.1246 90)
 			(effects
@@
 			)
 		)
-		(property "Value" "WS2812B"
+		(property "Value" "LED"
 			(at 243.84 39.0046 90)
 			(effects
@@
 			)
 		)
-		(property "Value" "WS2812B"
+		(property "Value" "LED"
 			(at 220.98 92.3446 90)
 			(effects
@@
 			)
 		)
-		(property "Value" "WS2812B"
+		(property "Value" "LED"
 			(at 267.97 74.5646 90)
 			(effects
@@
 			)
 		)
-		(property "Value" "WS2812B"
+		(property "Value" "LED"
 			(at 267.97 92.3446 90)
 			(effects
@@
 			)
 		)
-		(property "Value" "WS2812B"
+		(property "Value" "LED"
 			(at 267.97 39.0046 90)
 			(effects
@@
 			)
 		)
-		(property "Value" "120 pF"
+		(property "Value" "120pF"
 			(at 259.588 143.256 0)
 			(effects
@@
 			)
 		)
-		(property "Value" "WS2812B"
+		(property "Value" "LED"
 			(at 243.84 92.3446 90)
 			(effects

Commit message: Reverse LED data bus direction.
Parts:
- D10, D11, D12, D13, D14, D15, D16, D2, D3, D4, D5, D6, D7, D8, D9: footprint LED_SMD:LED_Wurth_150044M155260 -> LED_LTST:LED_LTST-E133CEGBK; symbol LED:WS2812B -> LED_LTST:LTST-E133CEGBK
Connections:
- net 2.7VCC: now also C13.1; no longer C13.2
- net GND: now also C13.2; no longer C13.1
- net at D9.2 (DIN): now also D8.4 (DOUT); no longer D10.4 (DIN)
- net at D9.4 (DOUT): now also D10.2 (DIN); no longer D8.2 (DOUT)
- net at D15.2 (DIN): now also D14.4 (DOUT); no longer D16.4 (DIN)
- net at D15.4 (DOUT): now also D16.2 (DIN); no longer D14.2 (DOUT)
- net at D12.2 (DIN): now also D11.4 (DOUT); no longer D13.4 (DIN)
- net at D12.4 (DOUT): now also D13.2 (DIN); no longer D11.2 (DOUT)
- net at C18.2, R1.2: now also D2.2 (DIN); no longer D2.4 (DIN)
- net at D5.2 (DIN): now also D4.4 (DOUT); no longer D6.4 (DIN)
- net at D5.4 (DOUT): now also D6.2 (DIN); no longer D4.2 (DOUT)
- net at D3.4 (DOUT): now also D4.2 (DIN); no longer D2.2 (DOUT)
- net at D7.2 (DIN): now also D6.4 (DOUT); no longer D8.4 (DIN)
- net at D7.4 (DOUT): now also D8.2 (DIN); no longer D6.2 (DOUT)
- net at D3.2 (DIN): now also D2.4 (DOUT); no longer D4.4 (DIN)
- new net: D10.4 (DOUT), D11.2 (DIN)
- new net: D13.4 (DOUT), D14.2 (DIN)
Other:
- moved on the sheet: C13
